File: ulx3s.kicad_pcb (KiCad board)
At the start: 4 copper layers, 94 x 50.8 mm, 235 parts, among them J1 CONN_02X20, J2 CONN_02X20, J3 WIFI_OFF, J4 CONN_02X03, J5 VJ1, Q1 BC857, Q2 2N7002, SW1 SW_DIP_x04, U1 LFE5U-85F-6BG381C, U10 IS25LP128F-JBLE, U11 PCA9306D, U2 MT48LC16M16A2TG, U3 TLV62569DBV, U4 TLV62569DBV, U5 TLV62569DBV, U6 FT231XQ, U7 MCP7940NT, U8 MAX11125, U9 ESP32, Y1 FNETHE025, Y2 32768Hz

Commit message: Initial draft
Parts:
- removed AUDIO1: JACK_TRS_6PINS, audio-jack:CUI_SJ-43516-SMT
- removed B1, B2, B3, B4, B5, B6: PTS645, Button_Switch_SMD:SW_SPST_PTS645
- removed C18: 100pF, Capacitor_SMD:C_0603_1608Metric
- removed C38, C39, C40, C41, C42, C43, C44, C45, C63, C64, C65, C66, C67, C68, C69, C70, C71, C72: 22nF, Capacitor_SMD:C_0603_1608Metric
- removed C46: 2.2uF, Capacitor_SMD:C_0805_2012Metric
- removed C58, C61: 22uF, Capacitor_SMD:C_0805_2012Metric
- removed C59, C62: 220nF, Capacitor_SMD:C_0603_1608Metric
- removed D&M: dm2mm, dm:dm2mm
- removed D0, D19, D4: RED, LED_SMD:LED_0805_2012Metric
- removed D1, D5: ORANGE, LED_SMD:LED_0805_2012Metric
- removed D18, D2, D6: GREEN, LED_SMD:LED_0805_2012Metric
- removed D22, D3, D7: BLUE, LED_SMD:LED_0805_2012Metric
- removed D30: 3.6V, Diode_SMD:D_SOD-323_HandSoldering
- removed D51, D52: 0, jumper:D_SMA_Jumper_NC
- removed EMARD (x2): emard12mm, emard:emard12mm
- removed GPDI1: GPDI-D, conn-fci:CONN-10029449-111RLF
- removed HR: HR, hrvatski_proizvod_veci:hrvatski
- removed J1, J2: CONN_02X20, Socket_Strips:Socket_Strip_Angled_2x20
- removed L4, L5: 33uH, Inductor_SMD:L_0805_2012Metric_Pad1.15x1.40mm_HandSolder
- removed LCD1: ST7789, st7789:st7789
- removed OSHW: OSHW2mm, oshw:oshw
- removed R14, R18, R57: 1.1k, Resistor_SMD:R_0603_1608Metric
- removed R15, R19, R36, R37, R41, R42, R43, R44, R45, R46, R47, R48, R58, R61, R62, R67: 549, Resistor_SMD:R_0603_1608Metric
- removed R16, R20, R59: 270, Resistor_SMD:R_0603_1608Metric
- removed R17, R21, R39, R51, R60, R7: 130, Resistor_SMD:R_0603_1608Metric
- removed R22, R23: 3.3k, Resistor_SMD:R_0603_1608Metric
- removed R24: 100k, Resistor_SMD:R_0603_1608Metric
- removed R25, R26: 4.7k, Resistor_SMD:R_0603_1608Metric
- removed R55: 10k, Resistor_SMD:R_0603_1608Metric
- removed REF**: inem, inem:inem
- removed SW1: SW_DIP_x04, dipswitch:SW_DIP_x4_W8.61mm_Slide_LowProfile
- removed U11: PCA9306D, SM8:SM8
- removed U8: MAX11125, max1112x-tqfn28:MAX1112x-TQFN-28-1EP_5x5mm_Pitch0.5mm
- removed fer: fer, fer:fer4mm6
- removed koncar: koncar, koncar:koncar
- removed radiona: radiona, radiona:radiona
Connections:
- SD1 pad 10: Net-(SD1-Pad10) -> unconnected-(SD1-SW-2-Pad10)
- SD1 pad 11: Net-(SD1-Pad11) -> unconnected-(SD1-NC-Pad11)
- SD1 pad 12: Net-(SD1-Pad12) -> unconnected-(SD1-NC-Pad12)
- U1 pad A10: GP1 -> (no net)
- U1 pad A11: GN1 -> (no net)
- U1 pad A12: FPDI_D2+ -> (no net)
- U1 pad A13: FPDI_D2- -> (no net)
- U1 pad A14: FPDI_D1+ -> (no net)
- U1 pad A15: Net-(U1-PadA15) -> (no net)
- U1 pad A16: FPDI_D0+ -> (no net)
- U1 pad A17: FPDI_CLK+ -> (no net)
- U1 pad A18: FPDI_CEC -> (no net)
- U1 pad A19: FPDI_UTIL -> (no net)
- U1 pad A2: GP9 -> (no net)
- U1 pad A3: AUDIO_R0 -> (no net)
- U1 pad A4: GP8 -> (no net)
- U1 pad A5: GN8 -> (no net)
- U1 pad A6: GP7 -> (no net)
- U1 pad A7: GP4 -> (no net)
- U1 pad A8: GN4 -> (no net)
- U1 pad A9: GP2 -> (no net)
- U1 pad B1: GN9 -> (no net)
- U1 pad B10: GN2 -> (no net)
- U1 pad B11: GP0 -> (no net)
- U1 pad B12: USB_FPGA_PULL_D+ -> (no net)
- U1 pad B13: GP26 -> (no net)
- U1 pad B15: GP22 -> (no net)
- U1 pad B16: FPDI_D0- -> (no net)
- U1 pad B17: GP23 -> (no net)
- U1 pad B18: FPDI_CLK- -> (no net)
- U1 pad B19: FPDI_SDA -> (no net)
- U1 pad B2: LED0 -> (no net)
- U1 pad B20: FPDI_HPD -> (no net)
- U1 pad B3: AUDIO_L3 -> (no net)
- U1 pad B4: GN10 -> (no net)
- U1 pad B5: AUDIO_R1 -> (no net)
- U1 pad B6: GN7 -> (no net)
- U1 pad B8: GN5 -> (no net)
- U1 pad B9: GP3 -> (no net)
- U1 pad C1: LED2 -> (no net)
- U1 pad C10: GN3 -> (no net)
- U1 pad C11: GN0 -> (no net)
- U1 pad C12: USB_FPGA_PULL_D- -> (no net)
- U1 pad C13: GN26 -> (no net)
- U1 pad C14: FPDI_D1- -> (no net)
- U1 pad C15: GN22 -> (no net)
- U1 pad C16: GP24 -> (no net)
- U1 pad C17: GN23 -> (no net)
- U1 pad C2: LED1 -> (no net)
- U1 pad C3: AUDIO_L2 -> (no net)
- U1 pad C4: GP10 -> (no net)
- U1 pad C5: AUDIO_R3 -> (no net)
- U1 pad C6: GP6 -> (no net)
- U1 pad C7: GN6 -> (no net)
- U1 pad C8: GP5 -> (no net)
- U1 pad C9: Net-(U1-PadC9) -> (no net)
- U1 pad D1: LED4 -> (no net)
- U1 pad D10: Net-(U1-PadD10) -> (no net)
- U1 pad D11: Net-(U1-PadD11) -> (no net)
- U1 pad D12: Net-(U1-PadD12) -> (no net)
- U1 pad D13: GP27 -> (no net)
- U1 pad D14: GP25 -> (no net)
- U1 pad D15: USB_FPGA_D+ -> (no net)
- U1 pad D16: GN24 -> (no net)
- U1 pad D2: LED3 -> (no net)
- U1 pad D3: AUDIO_L1 -> (no net)
- U1 pad D5: AUDIO_R2 -> (no net)
- U1 pad D6: BTN_PWRn -> (no net)
- U1 pad D7: SW3 -> (no net)
- U1 pad D8: SW2 -> (no net)
- U1 pad D9: Net-(U1-PadD9) -> (no net)
- U1 pad E1: LED6 -> (no net)
- U1 pad E10: Net-(U1-PadE10) -> (no net)
- U1 pad E11: Net-(U1-PadE11) -> (no net)
- U1 pad E12: FPDI_SCL -> (no net)
- U1 pad E13: GN27 -> (no net)
- U1 pad E14: GN25 -> (no net)
- U1 pad E15: USB_FPGA_D- -> (no net)
- U1 pad E2: LED5 -> (no net)
- U1 pad E3: GN11 -> (no net)
- U1 pad E4: AUDIO_L0 -> (no net)
- U1 pad E5: AUDIO_V3 -> (no net)
- U1 pad E6: WIFI_GPIO35 -> (no net)
- U1 pad E7: SW4 -> (no net)
- U1 pad E8: SW1 -> (no net)
- U1 pad E9: WIFI_GPIO25 -> (no net)
- U1 pad F2: AUDIO_V1 -> (no net)
- U1 pad F3: GN12 -> (no net)
- U1 pad F4: GP11 -> (no net)
- U1 pad F5: AUDIO_V2 -> (no net)
- U1 pad G3: GP12 -> (no net)
- U1 pad G5: GN13 -> (no net)
- U1 pad H3: LED7 -> (no net)
- U1 pad H4: GP13 -> (no net)
- U1 pad H5: AUDIO_V0 -> (no net)
- U1 pad K16: Net-(U1-PadK16) -> unconnected-(U1C-PR29A-PadK16)
- U1 pad K17: Net-(U1-PadK17) -> unconnected-(U1C-PR29B-PadK17)
- U1 pad M5: Net-(U1-PadM5) -> unconnected-(U1E-PL77A-PadM5)
- U1 pad R3: Net-(U1-PadR3) -> unconnected-(U1G-DOUT/CSOn-PadR3)
- U1 pad T10: +1V1 -> (no net)
- U1 pad T11: +1V1 -> (no net)
- U1 pad T12: +1V1 -> (no net)
- U1 pad T13: +1V1 -> (no net)
- U1 pad T14: +1V1 -> (no net)
- U1 pad T15: +1V1 -> (no net)
- U1 pad T16: Net-(U1-PadT16) -> unconnected-(U1D-PR77A-PadT16)
- U1 pad T6: +1V1 -> (no net)
- U1 pad T7: +1V1 -> (no net)
- U1 pad T8: +1V1 -> (no net)
- U1 pad T9: +1V1 -> (no net)
- U1 pad U15: +1V1 -> (no net)
- U1 pad U6: +1V1 -> (no net)
- U1 pad V10: +2V5 -> (no net)
- U1 pad V11: +2V5 -> (no net)
- U1 pad V17: +2V5 -> (no net)
- U1 pad V18: +2V5 -> (no net)
- U1 pad W13: Net-(U1-PadW13) -> (no net)
- U1 pad W14: Net-(U1-PadW14) -> (no net)
- U1 pad W17: /serdes/STXP11 -> (no net)
- U1 pad W18: /serdes/STXN11 -> (no net)
- U1 pad W20: Net-(U1-PadW20) -> (no net)
- U1 pad W4: Net-(U1-PadW4) -> (no net)
- U1 pad W5: Net-(U1-PadW5) -> (no net)
- U1 pad W8: Net-(U1-PadW8) -> (no net)
- U1 pad W9: Net-(U1-PadW9) -> (no net)
- U1 pad Y11: /serdes/SRCLKP -> (no net)
- U1 pad Y12: /serdes/SRCLKN -> (no net)
- U1 pad Y14: /serdes/SRXP10 -> (no net)
- U1 pad Y15: /serdes/SRXN10 -> (no net)
- U1 pad Y16: Net-(U1-PadY16) -> (no net)
- U1 pad Y17: Net-(U1-PadY17) -> (no net)
- U1 pad Y19: Net-(U1-PadY19) -> (no net)
- U1 pad Y5: /serdes/SRXP00 -> (no net)
- U1 pad Y6: /serdes/SRXN00 -> (no net)
- U1 pad Y7: /serdes/SRXP01 -> (no net)
- U1 pad Y8: /serdes/SRXN01 -> (no net)
- U9 pad 27: Net-(U9-Pad27) -> unconnected-(U9-IO16-Pad27)
- U9 pad 28: Net-(U9-Pad28) -> unconnected-(U9-IO17-Pad28)
- U9 pad 32: Net-(U9-Pad32) -> unconnected-(U9-NC-Pad32)
- US1 pad 4: Net-(US1-Pad4) -> unconnected-(US1-ID-Pad4)
- Y1 pad 2: GND -> +3V3
- Y2 pad 2: Net-(Y2-Pad2) -> unconnected-(Y2-G-Pad2)_1
- Y2 pad 3: Net-(Y2-Pad3) -> unconnected-(Y2-G-Pad2)
Routing:
- net (no net): track 0.00 -> 2754.1 mm, vias 0 -> 111
- net /blinkey/BTNPUR: track 76.6 -> 0.00 mm, vias 3 -> 0
- net GP27: track 57.4 -> 0.00 mm, vias 2 -> 0
- net GN27: track 56.8 -> 0.00 mm, vias 2 -> 0
- net GP0: track 54.6 -> 0.00 mm, vias 1 -> 0
- net GP1: track 53.5 -> 0.00 mm, vias 1 -> 0
- net GN0: track 53.4 -> 0.00 mm, vias 1 -> 0
- net GP25: track 53.0 -> 0.00 mm, vias 1 -> 0
- net GP26: track 53.0 -> 0.00 mm, vias 1 -> 0
- net GN26: track 52.9 -> 0.00 mm, vias 1 -> 0
- net GP24: track 52.3 -> 0.00 mm, vias 2 -> 0
- net GN25: track 51.8 -> 0.00 mm, vias 2 -> 0
- net GP2: track 50.9 -> 0.00 mm, vias 1 -> 0
- net GN1: track 50.5 -> 0.00 mm, vias 1 -> 0
- net GP3: track 50.1 -> 0.00 mm, vias 1 -> 0
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