File: wifi.kicad_sch (KiCad schematic)
At the start: 9 parts, among them J3 WIFI_OFF, U9 ESP32

Commit message: Initial draft
Other:
- company: EMARD -> (none)
- title: ULX3S -> FPGA CAM LCD
Changed lines of the file:
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@@
 	(generator "eeschema")
 	(generator_version "10.0")
-	(paper "A4")
+	(paper "B")
 	(title_block
-		(title "ULX3S")
-		(rev "1.0.9")
-		(company "EMARD")
-		(comment 1 "WIFI module ESP32")
+		(title "FPGA CAM LCD")
+		(date "2026-10-29")
+		(rev "0.1")
 	)
 	(text "TDO <v3.1"
@@
 		)
 		(instances
-			(project "ulx3s"
+			(project "FCL"
 				(path "/4fa0b2cb-19ee-4a85-acaa-86cc12a69b3d/00000000-0000-0000-0000-000058d6d447"
 					(reference "U9")
@@
 		)
 		(instances
-			(project "ulx3s"
+			(project "FCL"
 				(path "/4fa0b2cb-19ee-4a85-acaa-86cc12a69b3d/00000000-0000-0000-0000-000058d6d447"
 					(reference "#PWR0120")
@@
 		)
 		(instances
-			(project "ulx3s"
+			(project "FCL"
 				(path "/4fa0b2cb-19ee-4a85-acaa-86cc12a69b3d/00000000-0000-0000-0000-000058d6d447"
 					(reference "#PWR0119")
@@
 		)
 		(instances
-			(project "ulx3s"
+			(project "FCL"
 				(path "/4fa0b2cb-19ee-4a85-acaa-86cc12a69b3d/00000000-0000-0000-0000-000058d6d447"
 					(reference "#PWR0117")
@@
 		)
 		(instances
-			(project "ulx3s"
+			(project "FCL"
 				(path "/4fa0b2cb-19ee-4a85-acaa-86cc12a69b3d/00000000-0000-0000-0000-000058d6d447"
 					(reference "R34")
@@
 		)
 		(instances
-			(project "ulx3s"
+			(project "FCL"
 				(path "/4fa0b2cb-19ee-4a85-acaa-86cc12a69b3d/00000000-0000-0000-0000-000058d6d447"
 					(reference "#PWR0118")
@@
 		)
 		(instances
-			(project "ulx3s"
+			(project "FCL"
 				(path "/4fa0b2cb-19ee-4a85-acaa-86cc12a69b3d/00000000-0000-0000-0000-000058d6d447"
 					(reference "J3")
@@
 		)
 		(instances
-			(project "ulx3s"
+			(project "FCL"
 				(path "/4fa0b2cb-19ee-4a85-acaa-86cc12a69b3d/00000000-0000-0000-0000-000058d6d447"
 					(reference "R35")
@@
 		)
 		(instances
-			(project "ulx3s"
+			(project "FCL"
 				(path "/4fa0b2cb-19ee-4a85-acaa-86cc12a69b3d/00000000-0000-0000-0000-000058d6d447"
 					(reference "C21")
@@
 		)
 		(instances
-			(project "ulx3s"
+			(project "FCL"
 				(path "/4fa0b2cb-19ee-4a85-acaa-86cc12a69b3d/00000000-0000-0000-0000-000058d6d447"
 					(reference "#PWR0115")
@@
 		)
 		(instances
-			(project "ulx3s"
+			(project "FCL"
 				(path "/4fa0b2cb-19ee-4a85-acaa-86cc12a69b3d/00000000-0000-0000-0000-000058d6d447"
 					(reference "#PWR0116")
@@
 		)
 		(instances
-			(project "ulx3s"
+			(project "FCL"
 				(path "/4fa0b2cb-19ee-4a85-acaa-86cc12a69b3d/00000000-0000-0000-0000-000058d6d447"
 					(reference "#PWR0123")
@@
 		)
 		(instances
-			(project "ulx3s"
+			(project "FCL"
 				(path "/4fa0b2cb-19ee-4a85-acaa-86cc12a69b3d/00000000-0000-0000-0000-000058d6d447"
 					(reference "#PWR0121")
@@
 		)
 		(instances
-			(project "ulx3s"
+			(project "FCL"
 				(path "/4fa0b2cb-19ee-4a85-acaa-86cc12a69b3d/00000000-0000-0000-0000-000058d6d447"
 					(reference "#PWR0146")
@@
 		)
 		(instances
-			(project "ulx3s"
+			(project "FCL"
 				(path "/4fa0b2cb-19ee-4a85-acaa-86cc12a69b3d/00000000-0000-0000-0000-000058d6d447"
 					(reference "#PWR0148")
@@
 		)
 		(instances
-			(project "ulx3s"
+			(project "FCL"
 				(path "/4fa0b2cb-19ee-4a85-acaa-86cc12a69b3d/00000000-0000-0000-0000-000058d6d447"
 					(reference "R38")
@@
 		)
 		(instances
-			(project "ulx3s"
+			(project "FCL"
 				(path "/4fa0b2cb-19ee-4a85-acaa-86cc12a69b3d/00000000-0000-0000-0000-000058d6d447"
 					(reference "#PWR0149")
@@
 		)
 		(instances
-			(project "ulx3s"
+			(project "FCL"
 				(path "/4fa0b2cb-19ee-4a85-acaa-86cc12a69b3d/00000000-0000-0000-0000-000058d6d447"
 					(reference "C15")
@@
 		)
 		(instances
-			(project "ulx3s"
+			(project "FCL"
 				(path "/4fa0b2cb-19ee-4a85-acaa-86cc12a69b3d/00000000-0000-0000-0000-000058d6d447"
 					(reference "#PWR0150")
@@
 		)
 		(instances
-			(project "ulx3s"
+			(project "FCL"
 				(path "/4fa0b2cb-19ee-4a85-acaa-86cc12a69b3d/00000000-0000-0000-0000-000058d6d447"
 					(reference "SD1")
@@
 		)
 		(instances
-			(project "ulx3s"
+			(project "FCL"
 				(path "/4fa0b2cb-19ee-4a85-acaa-86cc12a69b3d/00000000-0000-0000-0000-000058d6d447"
 					(reference "#PWR043")
@@
 		)
 		(instances
-			(project "ulx3s"
+			(project "FCL"
 				(path "/4fa0b2cb-19ee-4a85-acaa-86cc12a69b3d/00000000-0000-0000-0000-000058d6d447"
 					(reference "R56")
