File: power.kicad_sch (KiCad schematic)
At the start: 84 parts, among them J5 VJ1, Q1 BC857, Q2 2N7002, U1 LFE5U-85F-6BG381C, U3 TLV62569DBV, U4 TLV62569DBV, U5 TLV62569DBV, U7 MCP7940NT, Y2 32768Hz

Commit message: Initial draft
Other:
- company: EMARD -> (none)
- title: ULX3S -> FPGA CAM LCD
