File: FCL.kicad_sch (KiCad schematic)
At the start: 4 parts

Commit message: Initial draft
Other:
- company: EMARD -> (none)
- title: ULX3S -> FPGA CAM LCD
Changed lines of the file:
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@@
 	(generator "eeschema")
 	(generator_version "10.0")
-	(paper "A4")
+	(paper "B")
 	(title_block
-		(title "ULX3S")
-		(rev "3.1.7")
-		(company "EMARD")
-		(comment 1 "Root sheet")
+		(title "FPGA CAM LCD")
+		(date "2026-10-29")
+		(rev "0.1")
 	)
 	(text "click on mouse pointer arrow on top of right toolbar\nand double-click on sheet to open"
@@
 		)
 		(instances
-			(project "ulx3s"
+			(project "FCL"
 				(path "/4fa0b2cb-19ee-4a85-acaa-86cc12a69b3d"
 					(reference "H1")
@@
 		)
 		(instances
-			(project "ulx3s"
+			(project "FCL"
 				(path "/4fa0b2cb-19ee-4a85-acaa-86cc12a69b3d"
 					(reference "H2")
@@
 		)
 		(instances
-			(project "ulx3s"
+			(project "FCL"
 				(path "/4fa0b2cb-19ee-4a85-acaa-86cc12a69b3d"
 					(reference "H3")
@@
 		)
 		(instances
-			(project "ulx3s"
+			(project "FCL"
 				(path "/4fa0b2cb-19ee-4a85-acaa-86cc12a69b3d"
 					(reference "H4")
@@
 		)
 		(instances
-			(project "ulx3s"
+			(project "FCL"
 				(path "/4fa0b2cb-19ee-4a85-acaa-86cc12a69b3d"
 					(reference "#PWR02")
@@
 		)
 		(instances
-			(project "ulx3s"
+			(project "FCL"
 				(path "/4fa0b2cb-19ee-4a85-acaa-86cc12a69b3d"
 					(reference "#PWR04")
@@
 		)
 		(instances
-			(project "ulx3s"
+			(project "FCL"
 				(path "/4fa0b2cb-19ee-4a85-acaa-86cc12a69b3d"
 					(reference "#PWR03")
@@
 		)
 		(instances
-			(project "ulx3s"
+			(project "FCL"
 				(path "/4fa0b2cb-19ee-4a85-acaa-86cc12a69b3d"
 					(reference "#PWR01")
@@
 		)
 		(instances
-			(project "ulx3s"
+			(project "FCL"
 				(path "/4fa0b2cb-19ee-4a85-acaa-86cc12a69b3d"
 					(page "2")
@@
 		)
 		(instances
-			(project "ulx3s"
+			(project "FCL"
 				(path "/4fa0b2cb-19ee-4a85-acaa-86cc12a69b3d"
 					(page "4")
@@
 		)
 		(instances
-			(project "ulx3s"
+			(project "FCL"
 				(path "/4fa0b2cb-19ee-4a85-acaa-86cc12a69b3d"
 					(page "9")
@@
 		)
 		(instances
-			(project "ulx3s"
+			(project "FCL"
 				(path "/4fa0b2cb-19ee-4a85-acaa-86cc12a69b3d"
 					(page "8")
@@
 		)
 		(instances
-			(project "ulx3s"
+			(project "FCL"
 				(path "/4fa0b2cb-19ee-4a85-acaa-86cc12a69b3d"
 					(page "11")

Commit message: initial draft start adding camera
Other:
- added sheet Camera (Camera.kicad_sch)
Changed lines of the file:
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@@
+		)
+	)
+	(sheet
+		(at 177.8 149.86)
+		(size 19.05 11.43)
+		(exclude_from_sim no)
+		(in_bom yes)
+		(on_board yes)
+		(dnp no)
+		(fields_autoplaced yes)
+		(stroke
+			(width 0)
+			(type solid)
+		)
+		(fill
+			(color 0 0 0 0)
+		)
+		(property "Sheetname" "Camera"
+			(at 177.8 149.0214 0)
+			(show_name no)
+			(do_not_autoplace no)
+			(effects
+				(font
+					(size 1.524 1.524)
+				)
+				(justify left bottom)
+			)
+		)
+		(property "Sheetfile" "Camera.kicad_sch"
+			(at 177.8 161.9762 0)
+			(show_name no)
+			(do_not_autoplace no)
+			(effects
+				(font
+					(size 1.524 1.524)
+				)
+				(justify left top)
+			)
+		)
+		(instances
+			(project "FCL"
+				(path "/4fa0b2cb-19ee-4a85-acaa-86cc12a69b3d"
+					(page "3")
+				)
+			)
 		)
 	)

Commit message: AI 1st attempt at add camera.
Other:
- sheet Camera ports: added CAM_D0, CAM_D1, CAM_D2, CAM_D3, CAM_D4, CAM_D5, CAM_D6, CAM_D7, CAM_HREF, CAM_PCLK, CAM_PWDN, CAM_RESETn, CAM_SIOC, CAM_SIOD, CAM_VSYNC, CAM_XCLK; removed none

Commit message: returned gpio.kicad_sch
Other:
- added sheet gpio (gpio.kicad_sch)
Changed lines of the file:
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@@
+	)
+	(sheet
+		(at 220.98 133.35)
+		(size 19.05 11.43)
+		(exclude_from_sim no)
+		(in_bom yes)
+		(on_board yes)
+		(dnp no)
+		(fields_autoplaced yes)
+		(stroke
+			(width 0)
+			(type solid)
+		)
+		(fill
+			(color 0 0 0 0)
+		)
+		(property "Sheetname" "gpio"
+			(at 220.98 132.5114 0)
+			(show_name no)
+			(do_not_autoplace no)
+			(effects
+				(font
+					(size 1.524 1.524)
+				)
+				(justify left bottom)
+			)
+		)
+		(property "Sheetfile" "gpio.kicad_sch"
+			(at 220.98 145.4662 0)
+			(show_name no)
+			(do_not_autoplace no)
+			(effects
+				(font
+					(size 1.524 1.524)
+				)
+				(justify left top)
+			)
+		)
+		(instances
+			(project "FCL"
+				(path "/4fa0b2cb-19ee-4a85-acaa-86cc12a69b3d"
+					(page "5")
+				)
+			)
+		)
 	)
 	(sheet
